File: schematic/schematic.kicad_sch (KiCad schematic)
At the start: 0 parts

Commit message: schematic and then I started editing the code...
Parts:
- added A1: Arduino_Nano_ESP32, Module:Arduino_Nano, symbol MCU_Module:Arduino_Nano_ESP32
- added C1: 220μF, symbol Device:C
- added DS1: ~, symbol New_Library:oled_display_module
- added SW1: SW_Push, symbol Switch:SW_Push
Connections:
- new net: A1.5 (D2), SW1.2
- new net: A1.10 (D7), DS1.16 (RESET)
- new net: A1.6 (D3), DS1.4 (DC)
- new net: A1.7 (D4), DS1.7 (Data0)
- new net: A1.8 (D5), DS1.8 (Data1)
- new net: A1.9 (D6), DS1.15 (CS)
- new net +3.3V: A1.17 (3V3), A1.29 (GND), A1.4 (GND), C1.1, C1.2, DS1.1 (GND), DS1.2 (3VPowerIn), DS1.20 (FrameGND), SW1.1
