File: schematic/schematic.kicad_sch (KiCad schematic)
At the start: 6 parts, among them SW1 SW_Push

Commit message: restarting laptop
Parts:
- BT1: footprint (none) -> Battery:BatteryHolder_Keystone_2462_2xAA
- BZ1: footprint (none) -> Buzzer_Beeper:Buzzer_TDK_PS1240P02BT_D12.2mm_H6.5mm
- C2: footprint (none) -> Capacitor_SMD:C_0201_0603Metric
- DS1: footprint (none) -> Library:OLED_Graphic_Display_Kit_Adafruit
- SW1: footprint (none) -> Button_Switch_THT:SW_PUSH-12mm
Connections:
- net +10V renamed +BATT
Changed lines of the file:
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@@
 	(wire
 		(pts
-			(xy 222.25 45.72) (xy 222.25 50.8)
+			(xy 215.9 76.2) (xy 215.9 102.87)
 		)
 		(stroke
@@
 	(wire
 		(pts
-			(xy 215.9 76.2) (xy 215.9 102.87)
+			(xy 226.06 76.2) (xy 215.9 76.2)
 		)
 		(stroke
@@
 	(wire
 		(pts
-			(xy 226.06 76.2) (xy 215.9 76.2)
+			(xy 256.54 119.38) (xy 256.54 124.46)
 		)
 		(stroke
@@
 	(wire
 		(pts
-			(xy 256.54 119.38) (xy 256.54 124.46)
+			(xy 222.25 44.45) (xy 222.25 50.8)
 		)
 		(stroke
@@
 			)
 		)
-		(property "Footprint" ""
+		(property "Footprint" "Button_Switch_THT:SW_PUSH-12mm"
 			(at 189.23 43.18 0)
 			(effects
@@
 	)
 	(symbol
+		(lib_id "power:+BATT")
+		(at 270.51 119.38 0)
+		(unit 1)
+		(exclude_from_sim no)
+		(in_bom yes)
+		(on_board yes)
+		(dnp no)
+		(fields_autoplaced yes)
+		(property "Reference" "#PWR013"
+			(at 270.51 123.19 0)
+			(effects
+				(font
+					(size 1.27 1.27)
+				)
+				(hide yes)
+			)
+		)
+		(property "Value" "+BATT"
+			(at 270.51 114.3 0)
+			(effects
+				(font
+					(size 1.27 1.27)
+				)
+			)
+		)
+		(property "Footprint" ""
+			(at 270.51 119.38 0)
+			(effects
+				(font
+					(size 1.27 1.27)
+				)
+				(hide yes)
+			)
+		)
+		(property "Datasheet" ""
+			(at 270.51 119.38 0)
+			(effects
+				(font
+					(size 1.27 1.27)
+				)
+				(hide yes)
+			)
+		)
+		(property "Description" "Power symbol creates a global label with name \"+BATT\""
+			(at 270.51 119.38 0)
+			(effects
+				(font
+					(size 1.27 1.27)
+				)
+				(hide yes)
+			)
+		)
+		(pin "1"
+		)
+		(instances
+			(project ""
+				(path "/3a91534b-bac7-4c1d-abc4-f3e0f0feb066"
+					(reference "#PWR013")
+					(unit 1)
+				)
+			)
+		)
+	)
+	(symbol
 		(lib_id "power:+3.3V")
 		(at 175.26 44.45 0)
@@
 	)
 	(symbol
-		(lib_id "power:+10V")
-		(at 270.51 119.38 0)
-		(unit 1)
-		(exclude_from_sim no)
-		(in_bom yes)
-		(on_board yes)
-		(dnp no)
-		(fields_autoplaced yes)
-		(property "Reference" "#PWR011"
-			(at 270.51 123.19 0)
-			(effects
-				(font
-					(size 1.27 1.27)
-				)
-				(hide yes)
-			)
-		)
-		(property "Value" "+10V"
-			(at 270.51 114.3 0)
-			(effects
-				(font
-					(size 1.27 1.27)
-				)
-			)
-		)
-		(property "Footprint" ""
-			(at 270.51 119.38 0)
-			(effects
-				(font
-					(size 1.27 1.27)
-				)
-				(hide yes)
-			)
-		)
-		(property "Datasheet" ""
-			(at 270.51 119.38 0)
-			(effects
-				(font
-					(size 1.27 1.27)
-				)
-				(hide yes)
-			)
-		)
-		(property "Description" "Power symbol creates a global label with name \"+10V\""
-			(at 270.51 119.38 0)
-			(effects
-				(font
-					(size 1.27 1.27)
-				)
-				(hide yes)
-			)
-		)
-		(pin "1"
-		)
-		(instances
-			(project ""
-				(path "/3a91534b-bac7-4c1d-abc4-f3e0f0feb066"
-					(reference "#PWR011")
-					(unit 1)
-				)
-			)
-		)
-	)
-	(symbol
 		(lib_id "power:GND")
 		(at 243.84 102.87 0)
@@
 	)
 	(symbol
+		(lib_id "power:+BATT")
+		(at 222.25 44.45 0)
+		(unit 1)
+		(exclude_from_sim no)
+		(in_bom yes)
+		(on_board yes)
+		(dnp no)
+		(fields_autoplaced yes)
+		(property "Reference" "#PWR012"
+			(at 222.25 48.26 0)
+			(effects
+				(font
+					(size 1.27 1.27)
+				)
+				(hide yes)
+			)
+		)
+		(property "Value" "+BATT"
+			(at 222.25 39.37 0)
+			(effects
+				(font
+					(size 1.27 1.27)
+				)
+			)
+		)
+		(property "Footprint" ""
+			(at 222.25 44.45 0)
+			(effects
+				(font
+					(size 1.27 1.27)
+				)
+				(hide yes)
+			)
+		)
+		(property "Datasheet" ""
+			(at 222.25 44.45 0)
+			(effects
+				(font
+					(size 1.27 1.27)
+				)
+				(hide yes)
+			)
+		)
+		(property "Description" "Power symbol creates a global label with name \"+BATT\""
+			(at 222.25 44.45 0)
+			(effects
+				(font
+					(size 1.27 1.27)
+				)
+				(hide yes)
+			)
+		)
+		(pin "1"
+		)
+		(instances
+			(project ""
+				(path "/3a91534b-bac7-4c1d-abc4-f3e0f0feb066"
+					(reference "#PWR012")
+					(unit 1)
+				)
+			)
+		)
+	)
+	(symbol
 		(lib_id "Device:C_US")
 		(at 256.54 128.27 0)
@@
 			)
 		)
-		(property "Footprint" ""
+		(property "Footprint" "Capacitor_SMD:C_0201_0603Metric"
 			(at 256.54 128.27 0)
 			(effects
@@
 	)
 	(symbol
-		(lib_id "power:+10V")
-		(at 222.25 45.72 0)
-		(unit 1)
-		(exclude_from_sim no)
-		(in_bom yes)
-		(on_board yes)
-		(dnp no)
-		(fields_autoplaced yes)
-		(property "Reference" "#PWR012"
-			(at 222.25 49.53 0)
-			(effects
-				(font
-					(size 1.27 1.27)
-				)
-				(hide yes)
-			)
-		)
-		(property "Value" "+10V"
-			(at 222.25 40.64 0)
-			(effects
-				(font
-					(size 1.27 1.27)
-				)
-			)
-		)
-		(property "Footprint" ""
-			(at 222.25 45.72 0)
-			(effects
-				(font
-					(size 1.27 1.27)
-				)
-				(hide yes)
-			)
-		)
-		(property "Datasheet" ""
-			(at 222.25 45.72 0)
-			(effects
-				(font
-					(size 1.27 1.27)
-				)
-				(hide yes)
-			)
-		)
-		(property "Description" "Power symbol creates a global label with name \"+10V\""
-			(at 222.25 45.72 0)
-			(effects
-				(font
-					(size 1.27 1.27)
-				)
-				(hide yes)
-			)
-		)
-		(pin "1"
-		)
-		(instances
-			(project "schematic"
-				(path "/3a91534b-bac7-4c1d-abc4-f3e0f0feb066"
-					(reference "#PWR012")
-					(unit 1)
-				)
-			)
-		)
-	)
-	(symbol
 		(lib_id "power:GND")
 		(at 135.89 86.36 0)
@@
 			)
 		)
-		(property "Footprint" ""
+		(property "Footprint" "Library:OLED_Graphic_Display_Kit_Adafruit"
 			(at 156.21 91.44 0)
 			(effects
@@
 			)
 		)
-		(property "Footprint" ""
+		(property "Footprint" "Buzzer_Beeper:Buzzer_TDK_PS1240P02BT_D12.2mm_H6.5mm"
 			(at 217.805 102.87 90)
 			(effects
@@
 			)
 		)
-		(property "Footprint" ""
+		(property "Footprint" "Battery:BatteryHolder_Keystone_2462_2xAA"
 			(at 270.51 126.746 90)
 			(effects

Commit message: finished readme and pcb
Parts:
- C2: footprint Capacitor_SMD:C_0201_0603Metric -> Capacitor_THT:C_Radial_D5.0mm_H11.0mm_P2.00mm
Connections:
- net at A1.10 (D7): now also DS1.4 (DC); no longer DS1.16 (RESET)
- net at A1.6 (D3): now also DS1.16 (RESET); no longer DS1.4 (DC)
- net at A1.7 (D4): now also DS1.15 (CS); no longer DS1.7 (Data0)
- net at A1.9 (D6): now also DS1.7 (Data0); no longer DS1.15 (CS)
Changed lines of the file:
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@@
-	(wire
-		(pts
-			(xy 182.88 81.28) (xy 182.88 73.66)
-		)
-		(stroke
-			(width 0)
-			(type default)
-		)
-	)
 	(wire
 		(pts
@@
 	(wire
 		(pts
-			(xy 160.02 66.04) (xy 226.06 66.04)
-		)
-		(stroke
-			(width 0)
-			(type default)
-		)
-	)
-	(wire
-		(pts
 			(xy 256.54 132.08) (xy 256.54 137.16)
 		)
@@
 	(wire
 		(pts
-			(xy 160.02 81.28) (xy 160.02 66.04)
-		)
-		(stroke
-			(width 0)
-			(type default)
-		)
-	)
-	(wire
-		(pts
-			(xy 152.4 63.5) (xy 226.06 63.5)
-		)
-		(stroke
-			(width 0)
-			(type default)
-		)
-	)
-	(wire
-		(pts
-			(xy 180.34 81.28) (xy 180.34 71.12)
+			(xy 160.02 81.28) (xy 160.02 71.12)
+		)
+		(stroke
+			(width 0)
+			(type default)
+		)
+	)
+	(wire
+		(pts
+			(xy 180.34 66.04) (xy 180.34 81.28)
 		)
 		(stroke
@@
 	(wire
 		(pts
+			(xy 182.88 81.28) (xy 182.88 63.5)
+		)
+		(stroke
+			(width 0)
+			(type default)
+		)
+	)
+	(wire
+		(pts
 			(xy 261.62 50.8) (xy 265.43 50.8)
 		)
@@
 	(wire
 		(pts
-			(xy 182.88 73.66) (xy 226.06 73.66)
-		)
-		(stroke
-			(width 0)
-			(type default)
-		)
-	)
-	(wire
-		(pts
-			(xy 180.34 71.12) (xy 226.06 71.12)
+			(xy 180.34 66.04) (xy 226.06 66.04)
+		)
+		(stroke
+			(width 0)
+			(type default)
+		)
+	)
+	(wire
+		(pts
+			(xy 160.02 71.12) (xy 226.06 71.12)
 		)
 		(stroke
@@
 	(wire
 		(pts
+			(xy 152.4 73.66) (xy 226.06 73.66)
+		)
+		(stroke
+			(width 0)
+			(type default)
+		)
+	)
+	(wire
+		(pts
 			(xy 215.9 76.2) (xy 215.9 102.87)
 		)
@@
 	(wire
 		(pts
+			(xy 182.88 63.5) (xy 226.06 63.5)
+		)
+		(stroke
+			(width 0)
+			(type default)
+		)
+	)
+	(wire
+		(pts
 			(xy 222.25 44.45) (xy 222.25 50.8)
 		)
@@
 	(wire
 		(pts
+			(xy 152.4 73.66) (xy 152.4 81.28)
+		)
+		(stroke
+			(width 0)
+			(type default)
+		)
+	)
+	(wire
+		(pts
 			(xy 270.51 119.38) (xy 270.51 123.19)
 		)
@@
 		(pts
 			(xy 265.43 50.8) (xy 265.43 43.18)
-		)
-		(stroke
-			(width 0)
-			(type default)
-		)
-	)
-	(wire
-		(pts
-			(xy 152.4 81.28) (xy 152.4 63.5)
 		)
 		(stroke
@@
 			)
 		)
-		(property "Footprint" "Capacitor_SMD:C_0201_0603Metric"
+		(property "Footprint" "Capacitor_THT:C_Radial_D5.0mm_H11.0mm_P2.00mm"
 			(at 256.54 128.27 0)
 			(effects
