File: schematic/schematic.kicad_pcb (KiCad board)
At the start: 2 copper layers, 3 parts

Commit message: restarting laptop
Parts:
- removed REF**: C_0201_0603Metric, Capacitor_SMD:C_0201_0603Metric
- removed REF**: Buzzer_TDK_PS1240P02BT_D12.2mm_H6.5mm, Buzzer_Beeper:Buzzer_TDK_PS1240P02BT_D12.2mm_H6.5mm
- added BT1: Battery, Battery:BatteryHolder_Keystone_2462_2xAA, B.Cu at (221.1, 51.7)
- added BZ1: Buzzer, Buzzer_Beeper:Buzzer_TDK_PS1240P02BT_D12.2mm_H6.5mm, B.Cu at (219.8, 42.0)
- added DS1: ~, Library:OLED_Graphic_Display_Kit_Adafruit, F.Cu at (224.7, 82.3)
- added SW1: SW_Push, Button_Switch_THT:SW_PUSH-12mm, F.Cu at (225.9, 37.4)
- moved A1 84.6 mm to (240.7, 119.0), turned to -90 degrees
Connections:
- A1 pad 30: +10V -> +BATT
Routing:
- added copper zone on In1.Cu, net +3.3V
- added copper zone on In1.Cu, net +BATT
- added copper zone on In2.Cu, net GND
Other:
- board outline added: 44 x 112 mm
- copper layers 2 -> 4
